File: eagle/esp8266_network_speaker/esp8266_network_speaker.brd (EAGLE design)
At the start: 100 x 80 mm, 0 parts

Commit message: wip, nothing interesting to report
Parts:
- added U$1: ESP8266_ESP-12, ESP8266-ESP12:ESP8266-ESP12
- added U1: 23A1024-I/SN, 23A1024:SOIC127P600X175-8N
- added U2: TSR_1-2433, _traco_tsr-1:TSR-1
Connections:
- new net ESP12_SPI_CLK: U$1.13
- new net ESP12_SPI_CS: U$1.2
- new net ESP12_SPI_MISO: U$1.14
- new net ESP12_SPI_MOSI: U$1.15
- new net GND: U2.2
- new net N$1: U$1.3
- new net N$4: U1.8
- new net N$5: U1.3
- new net N$6: U1.5
- new net N$7: U1.7
- new net N$8: U1.4
- new net N$9: U1.2
- new net RAM_/CS: U$1.4, U1.1
- new net RAM_SCK: U1.6
- new net VO: U2.3
Changed lines of the file:
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@@
 <layer number="48" name="Document" color="7" fill="1" visible="yes" active="yes"/>
 <layer number="49" name="Reference" color="7" fill="1" visible="yes" active="yes"/>
+<layer number="50" name="dxf" color="7" fill="1" visible="yes" active="yes"/>
 <layer number="51" name="tDocu" color="7" fill="1" visible="yes" active="yes"/>
 <layer number="52" name="bDocu" color="7" fill="1" visible="yes" active="yes"/>
@@
 <layer number="97" name="Info" color="7" fill="1" visible="no" active="no"/>
 <layer number="98" name="Guide" color="6" fill="1" visible="no" active="no"/>
+<layer number="200" name="200bmp" color="7" fill="1" visible="yes" active="yes"/>
 </layers>
 <board>
@@
 </autorouter>
 <elements>
+<element name="U1" library="23A1024" package="SOIC127P600X175-8N" value="23A1024-I/SN" x="21.59" y="20.32">
+<attribute name="MPN" value="23A1024-I/SN" x="21.59" y="20.32" size="1.778" layer="27" display="off"/>
+<attribute name="PACKAGE" value="SOIC-8" x="21.59" y="20.32" size="1.778" layer="27" display="off"/>
+<attribute name="OC_FARNELL" value="2212147" x="21.59" y="20.32" size="1.778" layer="27" display="off"/>
+<attribute name="SUPPLIER" value="MICROCHIP" x="21.59" y="20.32" size="1.778" layer="27" display="off"/>
+<attribute name="OC_NEWARK" value="94T8191" x="21.59" y="20.32" size="1.778" layer="27" display="off"/>
+</element>
+<element name="U$1" library="ESP8266-ESP12" package="ESP8266-ESP12" value="ESP8266_ESP-12" x="17.78" y="24.13"/>
+<element name="U2" library="_traco_tsr-1" package="TSR-1" value="TSR_1-2433" x="33.02" y="16.51"/>
 </elements>
 <signals>
+<signal name="GND">
+<contactref element="U2" pad="2"/>
+</signal>
+<signal name="VO">
+<contactref element="U2" pad="3"/>
+</signal>
+<signal name="ESP12_SPI_MISO">
+<contactref element="U$1" pad="14"/>
+</signal>
+<signal name="ESP12_SPI_MOSI">
+<contactref element="U$1" pad="15"/>
+</signal>
+<signal name="ESP12_SPI_CLK">
+<contactref element="U$1" pad="13"/>
+</signal>
+<signal name="ESP12_SPI_CS">
+<contactref element="U$1" pad="2"/>
+</signal>
+<signal name="N$1">
+<contactref element="U$1" pad="3"/>
+</signal>
+<signal name="RAM_/CS">
+<contactref element="U$1" pad="4"/>
+<contactref element="U1" pad="1"/>
+<wire x1="19.2278" y1="22.225" x2="33.98" y2="32.13" width="0" layer="19" extent="1-1"/>
+</signal>
+<signal name="RAM_SCK">
+<contactref element="U1" pad="6"/>
+</signal>
+<signal name="N$4">
+<contactref element="U1" pad="8"/>
+</signal>
+<signal name="N$5">
+<contactref element="U1" pad="3"/>
+</signal>
+<signal name="N$6">
+<contactref element="U1" pad="5"/>
+</signal>
+<signal name="N$7">
+<contactref element="U1" pad="7"/>
+</signal>
+<signal name="N$8">
+<contactref element="U1" pad="4"/>
+</signal>
+<signal name="N$9">
+<contactref element="U1" pad="2"/>
+</signal>
 </signals>
 </board>
